File: RPiCluster2/RPiCluster2.kicad_pcb (KiCad board)
At the start: 2 copper layers, 100 x 100 mm, 88 parts, among them J1 RPi_slave_1, J10 Addr_1, J11 Addr_0, J2 RPi_slave_2, J3 RPi_slave_3, J4 RPi_slave_4, J5 Addr, J6 Power_header, J7 Signal_header, J8 Signal_socket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

Commit message: RPiCluster2: Update
Parts:
- removed C12, C13, C16, C17: 10u, Capacitor_THT:C_Rect_L7.2mm_W3.0mm_P5.00mm_FKS2_FKP2_MKS2_MKP2
- moved C15 26.9 mm to (126.4, 93.3), turned to 270 degrees
- moved R32 25.6 mm to (116.2, 86.4)
- moved D12 25.1 mm to (129.5, 101.6), turned to 180 degrees
- moved C14 24.5 mm to (118.7, 92.7), turned to 270 degrees
- moved D11 19.9 mm to (116.8, 101.6)
- moved R31 18.8 mm to (115.6, 89.5)
- moved Q7 5.23 mm to (130.6, 95.2)
- moved Q6 4.26 mm to (122.6, 95.0)
Routing:
- net SCL: track 17.1 -> 215.4 mm, vias 0 -> 1
- net SDA: track 21.4 -> 211.2 mm
- net TXD: track 6.13 -> 113.8 mm
- net RXD: track 6.77 -> 108.0 mm
- net GND: track 270.1 -> 364.0 mm
- net /TXD4: track 0.00 -> 55.8 mm, vias 0 -> 2
- net /RXD4: track 0.00 -> 52.3 mm, vias 0 -> 2
- net /TXD1: track 3.54 -> 55.2 mm
- net /TXD_SLV: track 3.81 -> 47.0 mm, vias 0 -> 2
- net /TXD3: track 0.00 -> 39.9 mm, vias 0 -> 2
- net /RXD1: track 3.67 -> 40.5 mm, vias 0 -> 1
- net +3V3: track 289.7 -> 324.9 mm
- net /TXD2: track 0.00 -> 29.7 mm, vias 0 -> 2
- net 5V_SLV3: track 0.00 -> 24.2 mm
- net +5V: track 43.4 -> 19.8 mm, vias 2 -> 56
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- added copper zone on B.Cu, net +5V
- added copper zone on B.Cu, net GND
- added copper zone on F.Cu, net GND

Commit message: RPiCluster2: Pass DRC
Parts:
- moved TP2 3.70 mm to (75.2, 108.7)
Routing:
- net GND: track 364.0 -> 709.5 mm
- net 5V_SLV1: track 31.3 -> 34.1 mm

Commit message: RPiCluster2: Bump to v0.0.0
Parts:
- added TMP: MountingHole_2.7mm_M2.5, MountingHole:MountingHole_2.7mm_M2.5, F.Cu at (130.3, 89.8)
Routing:
- net GND: track 709.5 -> 287.6 mm, vias 0 -> 308
Other:
- rule trace_min: 0.2 -> 0.25
- board text added: "RPiCluster2 v.0.0.0 (c) 2018 Sugizaki Yukimasa"
