File: Motherboard/Motherboard.kicad_pcb (KiCad board)
At the start: 2 copper layers, 100 x 100 mm, 2 parts

Commit message: Motherboard: Update
Parts:
- added C1: 10u, Capacitor_THT:C_Rect_L7.2mm_W3.0mm_P5.00mm_FKS2_FKP2_MKS2_MKP2, F.Cu at (104.1, 87.6)
- added C2: 10u, Capacitor_THT:C_Rect_L7.2mm_W3.0mm_P5.00mm_FKS2_FKP2_MKS2_MKP2, F.Cu at (104.1, 91.4)
- added C3: 470u, Capacitor_THT:CP_Radial_D10.0mm_P2.50mm_P5.00mm, F.Cu at (123.2, 85.1)
- added C4: 470u, Capacitor_THT:CP_Radial_D10.0mm_P2.50mm_P5.00mm, F.Cu at (134.3, 85.1)
- added C5: 10u, Capacitor_THT:CP_Radial_D5.0mm_P2.50mm, F.Cu at (124.5, 141.0)
- added C6: 10u, Capacitor_THT:C_Rect_L7.2mm_W3.0mm_P5.00mm_FKS2_FKP2_MKS2_MKP2, F.Cu at (116.8, 123.2)
- added C8: 10u, Capacitor_THT:C_Rect_L7.2mm_W3.0mm_P5.00mm_FKS2_FKP2_MKS2_MKP2, F.Cu at (69.9, 121.9)
- added D1: 0V5, Diode_THT:D_T-1_P5.08mm_Horizontal, F.Cu at (129.5, 130.8)
- added D2: 0V5, Diode_THT:D_T-1_P5.08mm_Horizontal, F.Cu at (121.9, 135.9)
- added D3: LED_power_down, LED_THT:LED_D3.0mm, F.Cu at (71.1, 85.1)
- added J1: Signal_socket, Connector_PinSocket_2.54mm:PinSocket_1x06_P2.54mm_Horizontal, F.Cu at (143.5, 134.6)
- added J2: ATX_power, Connector_Molex:Molex_Mini-Fit_Jr_5569-24A2_2x12_P4.20mm_Horizontal, F.Cu at (88.4, 64.8)
- added J3: RPi_server, Connector_PinSocket_2.54mm:PinSocket_2x20_P2.54mm_Vertical, F.Cu at (101.6, 95.2)
- added J4: Power_socket, Connector_PinSocket_2.54mm:PinSocket_2x20_P2.54mm_Horizontal, F.Cu at (142.2, 113.0)
- added J5: Test_~PS_ON~, Connector_PinHeader_2.54mm:PinHeader_1x02_P2.54mm_Vertical, F.Cu at (80.0, 124.5)
- added Q1: 2SA1015, Package_TO_SOT_THT:TO-92_Inline, F.Cu at (59.7, 85.1)
- added R1: 2k, Resistor_THT:R_Axial_DIN0207_L6.3mm_D2.5mm_P7.62mm_Horizontal, F.Cu at (127.0, 120.7)
- added R10: 10k±1%, Resistor_THT:R_Axial_DIN0207_L6.3mm_D2.5mm_P7.62mm_Horizontal, F.Cu at (59.7, 115.6)
- added R11: 10k±1%, Resistor_THT:R_Axial_DIN0207_L6.3mm_D2.5mm_P7.62mm_Horizontal, F.Cu at (82.5, 113.0)
- added R12: 10k, Resistor_THT:R_Axial_DIN0207_L6.3mm_D2.5mm_P7.62mm_Horizontal, F.Cu at (69.8, 105.4)
- added R2: 10k, Resistor_THT:R_Axial_DIN0207_L6.3mm_D2.5mm_P7.62mm_Horizontal, F.Cu at (121.9, 118.1)
- added R3: 47k, Resistor_THT:R_Axial_DIN0207_L6.3mm_D2.5mm_P7.62mm_Horizontal, F.Cu at (77.5, 108.0)
- added R4: 1k, Resistor_THT:R_Axial_DIN0207_L6.3mm_D2.5mm_P7.62mm_Horizontal, F.Cu at (66.0, 86.4)
- added R5: 6k8±5%, Resistor_THT:R_Axial_DIN0207_L6.3mm_D2.5mm_P7.62mm_Horizontal, F.Cu at (67.3, 105.4)
- added R6: 3k3±5%, Resistor_THT:R_Axial_DIN0207_L6.3mm_D2.5mm_P7.62mm_Horizontal, F.Cu at (62.2, 108.0)
- added R7: 3k3±5%, Resistor_THT:R_Axial_DIN0207_L6.3mm_D2.5mm_P7.62mm_Horizontal, F.Cu at (80.0, 105.4)
- added R8: 10k, Resistor_THT:R_Axial_DIN0207_L6.3mm_D2.5mm_P7.62mm_Horizontal, F.Cu at (61.0, 88.9)
- added R9: 10k±1%, Resistor_THT:R_Axial_DIN0207_L6.3mm_D2.5mm_P7.62mm_Horizontal, F.Cu at (64.8, 113.0)
- added SW1: Reset, Button_Switch_THT:SW_PUSH_6mm, F.Cu at (58.4, 97.8)
- added TP1: Test_VEE, Connector_PinHeader_2.54mm:PinHeader_1x02_P2.54mm_Vertical, F.Cu at (120.7, 143.5)
- added U1: LM358, Package_DIP:DIP-8_W7.62mm, F.Cu at (124.5, 125.7)
- added U2: ATtiny13A-PU, Package_DIP:DIP-8_W7.62mm, F.Cu at (69.8, 110.5)
Routing:
- net GND: track 0.00 -> 45.2 mm
- net +5VD: track 0.00 -> 17.6 mm
- net Net-(R1-Pad2): track 0.00 -> 17.3 mm
- net VEE: track 0.00 -> 15.8 mm
- net Net-(R10-Pad1): track 0.00 -> 10.2 mm
- net Net-(D1-Pad1): track 0.00 -> 9.72 mm
- net -12V: track 0.00 -> 8.67 mm
- net Net-(R5-Pad2): track 0.00 -> 5.08 mm
- net Net-(R11-Pad1): track 0.00 -> 5.08 mm
- net Net-(D2-Pad1): track 0.00 -> 5.08 mm
- net Net-(Q1-Pad3): track 0.00 -> 4.34 mm
- net Net-(Q1-Pad2): track 0.00 -> 3.81 mm
- net Net-(D3-Pad2): track 0.00 -> 3.81 mm
- net Net-(R12-Pad1): track 0.00 -> 2.54 mm
Other:
- net class Default: clearance 0.2 -> 0.25
- rule trace_clearance: 0.2 -> 0.25

Commit message: Motherboard: Update
Parts:
- added REF**: MountingHole_3.2mm_M3, MountingHole:MountingHole_3.2mm_M3, F.Cu at (53.8, 147.8)
- added REF**: MountingHole_2.7mm_M2.5_Pad_Via, MountingHole:MountingHole_2.7mm_M2.5_Pad_Via, F.Cu at (94.8, 89.8)
- added REF**: MountingHole_2.7mm_M2.5, MountingHole:MountingHole_2.7mm_M2.5, F.Cu at (94.8, 89.8)
- added REF**: MountingHole_3.2mm_M3_Pad_Via, MountingHole:MountingHole_3.2mm_M3_Pad_Via, F.Cu at (53.8, 147.8)
- added REF**: MountingHole_3.2mm_M3_Pad_Via, MountingHole:MountingHole_3.2mm_M3_Pad_Via, F.Cu at (147.8, 147.8)
- added REF**: MountingHole_3.2mm_M3, MountingHole:MountingHole_3.2mm_M3, F.Cu at (147.8, 147.8)
- added REF**: MountingHole_3.2mm_M3, MountingHole:MountingHole_3.2mm_M3, F.Cu at (147.8, 53.8)
- added REF**: MountingHole_3.2mm_M3_Pad_Via, MountingHole:MountingHole_3.2mm_M3_Pad_Via, F.Cu at (147.8, 53.8)
- added REF**: MountingHole_2.7mm_M2.5_Pad_Via, MountingHole:MountingHole_2.7mm_M2.5_Pad_Via, F.Cu at (94.8, 147.8)
- added REF**: MountingHole_2.7mm_M2.5, MountingHole:MountingHole_2.7mm_M2.5, F.Cu at (94.8, 147.8)
- moved TP1 31.4 mm to (142.2, 120.7), turned to 270 degrees
- moved C8 30.5 mm to (68.7, 91.4)
- moved R11 30.5 mm to (81.3, 82.5)
- moved R3 30.5 mm to (76.2, 77.5)
- moved R6 30.5 mm to (61.0, 77.5)
- moved R9 30.5 mm to (63.5, 82.5)
- moved SW1 30.5 mm to (57.1, 67.3)
- moved J5 30.5 mm to (78.7, 94.0)
- moved R10 30.5 mm to (58.4, 85.1)
- moved R12 30.5 mm to (68.6, 74.9)
- moved R5 30.5 mm to (66.0, 74.9)
- moved R7 30.5 mm to (78.7, 74.9)
- moved U2 30.5 mm to (68.6, 80.0)
- moved C5 28.5 mm to (139.7, 116.8), turned to 90 degrees
- moved D3 25.4 mm to (72.4, 59.7)
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Routing:
- net GND: track 45.2 -> 205.7 mm
- net +5V: track 0.00 -> 100.2 mm
- net /SDA: track 0.00 -> 72.9 mm, vias 0 -> 2
- net /SCL: track 0.00 -> 72.9 mm, vias 0 -> 2
- net /RXD: track 0.00 -> 70.5 mm
- net /TXD: track 0.00 -> 69.7 mm
- net /PWR_OK: track 0.00 -> 56.9 mm
- net /~PS_ON~: track 0.00 -> 39.0 mm
- net +3V3: track 0.00 -> 34.8 mm
- net Net-(R12-Pad2): track 0.00 -> 11.4 mm
- net Net-(R1-Pad2): track 17.3 -> 19.9 mm
- net Net-(R12-Pad1): track 2.54 -> 5.08 mm
- net -12V: track 8.67 -> 7.62 mm
- net VEE: track 15.8 -> 16.9 mm
- net Net-(D1-Pad1): track 9.72 -> 8.67 mm
- added copper zone on F.Cu, net GND

Commit message: Motherboard: Update
Parts:
- added REF**: SolderWirePad_1x01_Drill1mm, Connector_Wire:SolderWirePad_1x01_Drill1mm, F.Cu at (117.3, 140.2)
- added REF**: SolderWirePad_1x01_Drill1mm, Connector_Wire:SolderWirePad_1x01_Drill1mm, F.Cu at (130.0, 140.2)
- added REF**: SolderWirePad_1x01_Drill1mm, Connector_Wire:SolderWirePad_1x01_Drill1mm, F.Cu at (69.0, 119.9)
- added REF**: SolderWirePad_1x01_Drill1mm, Connector_Wire:SolderWirePad_1x01_Drill1mm, F.Cu at (61.4, 119.9)
- added REF**: SolderWirePad_1x01_Drill1mm, Connector_Wire:SolderWirePad_1x01_Drill1mm, F.Cu at (56.3, 119.9)
- added REF**: SolderWirePad_1x01_Drill1mm, Connector_Wire:SolderWirePad_1x01_Drill1mm, F.Cu at (64.0, 122.4)
- added REF**: SolderWirePad_1x01_Drill1mm, Connector_Wire:SolderWirePad_1x01_Drill1mm, F.Cu at (66.5, 122.4)
- added REF**: SolderWirePad_1x01_Drill1mm, Connector_Wire:SolderWirePad_1x01_Drill1mm, F.Cu at (69.0, 107.2)
- added REF**: SolderWirePad_1x01_Drill1mm, Connector_Wire:SolderWirePad_1x01_Drill1mm, F.Cu at (71.6, 104.6)
- added REF**: SolderWirePad_1x01_Drill1mm, Connector_Wire:SolderWirePad_1x01_Drill1mm, F.Cu at (56.3, 109.7)
- added REF**: SolderWirePad_1x01_Drill1mm, Connector_Wire:SolderWirePad_1x01_Drill1mm, F.Cu at (64.0, 114.8)
- added REF**: SolderWirePad_1x01_Drill1mm, Connector_Wire:SolderWirePad_1x01_Drill1mm, F.Cu at (74.1, 114.8)
- added REF**: SolderWirePad_1x01_Drill1mm, Connector_Wire:SolderWirePad_1x01_Drill1mm, F.Cu at (124.9, 140.2)
- added REF**: SolderWirePad_1x01_Drill1mm, Connector_Wire:SolderWirePad_1x01_Drill1mm, F.Cu at (61.4, 122.4)
- added REF**: SolderWirePad_1x01_Drill1mm, Connector_Wire:SolderWirePad_1x01_Drill1mm, F.Cu at (58.9, 122.4)
- added REF**: SolderWirePad_1x01_Drill1mm, Connector_Wire:SolderWirePad_1x01_Drill1mm, F.Cu at (69.0, 114.8)
- added REF**: SolderWirePad_1x01_Drill1mm, Connector_Wire:SolderWirePad_1x01_Drill1mm, F.Cu at (53.8, 119.9)
- added REF**: SolderWirePad_1x01_Drill1mm, Connector_Wire:SolderWirePad_1x01_Drill1mm, F.Cu at (76.7, 119.9)
- added REF**: SolderWirePad_1x01_Drill1mm, Connector_Wire:SolderWirePad_1x01_Drill1mm, F.Cu at (56.3, 122.4)
- added REF**: SolderWirePad_1x01_Drill1mm, Connector_Wire:SolderWirePad_1x01_Drill1mm, F.Cu at (64.0, 119.9)
- added REF**: SolderWirePad_1x01_Drill1mm, Connector_Wire:SolderWirePad_1x01_Drill1mm, F.Cu at (74.1, 119.9)
- added REF**: SolderWirePad_1x01_Drill1mm, Connector_Wire:SolderWirePad_1x01_Drill1mm, F.Cu at (66.5, 119.9)
- added REF**: SolderWirePad_1x01_Drill1mm, Connector_Wire:SolderWirePad_1x01_Drill1mm, F.Cu at (81.7, 107.2)
- added REF**: SolderWirePad_1x01_Drill1mm, Connector_Wire:SolderWirePad_1x01_Drill1mm, F.Cu at (140.2, 142.7)
- added REF**: SolderWirePad_1x01_Drill1mm, Connector_Wire:SolderWirePad_1x01_Drill1mm, F.Cu at (58.9, 104.6)
- added REF**: SolderWirePad_1x01_Drill1mm, Connector_Wire:SolderWirePad_1x01_Drill1mm, F.Cu at (81.7, 104.6)
- added REF**: SolderWirePad_1x01_Drill1mm, Connector_Wire:SolderWirePad_1x01_Drill1mm, F.Cu at (81.7, 112.2)
- added REF**: SolderWirePad_1x01_Drill1mm, Connector_Wire:SolderWirePad_1x01_Drill1mm, F.Cu at (69.0, 122.4)
- added REF**: SolderWirePad_1x01_Drill1mm, Connector_Wire:SolderWirePad_1x01_Drill1mm, F.Cu at (71.6, 119.9)
- added REF**: SolderWirePad_1x01_Drill1mm, Connector_Wire:SolderWirePad_1x01_Drill1mm, F.Cu at (71.6, 122.4)
- added REF**: SolderWirePad_1x01_Drill1mm, Connector_Wire:SolderWirePad_1x01_Drill1mm, F.Cu at (53.8, 122.4)
- added REF**: SolderWirePad_1x01_Drill1mm, Connector_Wire:SolderWirePad_1x01_Drill1mm, F.Cu at (79.2, 119.9)
- added REF**: SolderWirePad_1x01_Drill1mm, Connector_Wire:SolderWirePad_1x01_Drill1mm, F.Cu at (58.9, 119.9)
- added REF**: SolderWirePad_1x01_Drill1mm, Connector_Wire:SolderWirePad_1x01_Drill1mm, F.Cu at (81.7, 119.9)
- added REF**: SolderWirePad_1x01_Drill1mm, Connector_Wire:SolderWirePad_1x01_Drill1mm, F.Cu at (135.1, 142.7)
- added REF**: SolderWirePad_1x01_Drill1mm, Connector_Wire:SolderWirePad_1x01_Drill1mm, F.Cu at (69.0, 109.7)
- added REF**: SolderWirePad_1x01_Drill1mm, Connector_Wire:SolderWirePad_1x01_Drill1mm, F.Cu at (61.4, 109.7)
- added REF**: SolderWirePad_1x01_Drill1mm, Connector_Wire:SolderWirePad_1x01_Drill1mm, F.Cu at (61.4, 107.2)
- added REF**: SolderWirePad_1x01_Drill1mm, Connector_Wire:SolderWirePad_1x01_Drill1mm, F.Cu at (74.1, 117.3)
- added REF**: SolderWirePad_1x01_Drill1mm, Connector_Wire:SolderWirePad_1x01_Drill1mm, F.Cu at (74.1, 122.4)
- added REF**: SolderWirePad_1x01_Drill1mm, Connector_Wire:SolderWirePad_1x01_Drill1mm, F.Cu at (56.3, 114.8)
- added REF**: SolderWirePad_1x01_Drill1mm, Connector_Wire:SolderWirePad_1x01_Drill1mm, F.Cu at (64.0, 117.3)
- added REF**: SolderWirePad_1x01_Drill1mm, Connector_Wire:SolderWirePad_1x01_Drill1mm, F.Cu at (66.5, 117.3)
- added REF**: SolderWirePad_1x01_Drill1mm, Connector_Wire:SolderWirePad_1x01_Drill1mm, F.Cu at (61.4, 117.3)
- added REF**: SolderWirePad_1x01_Drill1mm, Connector_Wire:SolderWirePad_1x01_Drill1mm, F.Cu at (56.3, 112.2)
- added REF**: SolderWirePad_1x01_Drill1mm, Connector_Wire:SolderWirePad_1x01_Drill1mm, F.Cu at (137.6, 142.7)
- added REF**: SolderWirePad_1x01_Drill1mm, Connector_Wire:SolderWirePad_1x01_Drill1mm, F.Cu at (64.0, 109.7)
- added REF**: SolderWirePad_1x01_Drill1mm, Connector_Wire:SolderWirePad_1x01_Drill1mm, F.Cu at (61.4, 104.6)
- added REF**: SolderWirePad_1x01_Drill1mm, Connector_Wire:SolderWirePad_1x01_Drill1mm, F.Cu at (61.4, 114.8)
- added REF**: SolderWirePad_1x01_Drill1mm, Connector_Wire:SolderWirePad_1x01_Drill1mm, F.Cu at (66.5, 114.8)
- added REF**: SolderWirePad_1x01_Drill1mm, Connector_Wire:SolderWirePad_1x01_Drill1mm, F.Cu at (69.0, 117.3)
- added REF**: SolderWirePad_1x01_Drill1mm, Connector_Wire:SolderWirePad_1x01_Drill1mm, F.Cu at (71.6, 114.8)
- added REF**: SolderWirePad_1x01_Drill1mm, Connector_Wire:SolderWirePad_1x01_Drill1mm, F.Cu at (71.6, 117.3)
- added REF**: SolderWirePad_1x01_Drill1mm, Connector_Wire:SolderWirePad_1x01_Drill1mm, F.Cu at (53.8, 117.3)
- added REF**: SolderWirePad_1x01_Drill1mm, Connector_Wire:SolderWirePad_1x01_Drill1mm, F.Cu at (79.2, 117.3)
- added REF**: SolderWirePad_1x01_Drill1mm, Connector_Wire:SolderWirePad_1x01_Drill1mm, F.Cu at (74.1, 112.2)
- added REF**: SolderWirePad_1x01_Drill1mm, Connector_Wire:SolderWirePad_1x01_Drill1mm, F.Cu at (114.8, 142.7)
- added REF**: SolderWirePad_1x01_Drill1mm, Connector_Wire:SolderWirePad_1x01_Drill1mm, F.Cu at (56.3, 104.6)
- added REF**: SolderWirePad_1x01_Drill1mm, Connector_Wire:SolderWirePad_1x01_Drill1mm, F.Cu at (64.0, 107.2)
- added REF**: SolderWirePad_1x01_Drill1mm, Connector_Wire:SolderWirePad_1x01_Drill1mm, F.Cu at (66.5, 107.2)
- added REF**: SolderWirePad_1x01_Drill1mm, Connector_Wire:SolderWirePad_1x01_Drill1mm, F.Cu at (66.5, 104.6)
- added REF**: SolderWirePad_1x01_Drill1mm, Connector_Wire:SolderWirePad_1x01_Drill1mm, F.Cu at (58.9, 117.3)
- added REF**: SolderWirePad_1x01_Drill1mm, Connector_Wire:SolderWirePad_1x01_Drill1mm, F.Cu at (53.8, 114.8)
- added REF**: SolderWirePad_1x01_Drill1mm, Connector_Wire:SolderWirePad_1x01_Drill1mm, F.Cu at (76.7, 114.8)
- added REF**: SolderWirePad_1x01_Drill1mm, Connector_Wire:SolderWirePad_1x01_Drill1mm, F.Cu at (79.2, 112.2)
- added REF**: SolderWirePad_1x01_Drill1mm, Connector_Wire:SolderWirePad_1x01_Drill1mm, F.Cu at (74.1, 107.2)
- added REF**: SolderWirePad_1x01_Drill1mm, Connector_Wire:SolderWirePad_1x01_Drill1mm, F.Cu at (53.8, 109.7)
- added REF**: SolderWirePad_1x01_Drill1mm, Connector_Wire:SolderWirePad_1x01_Drill1mm, F.Cu at (132.6, 142.7)
- added REF**: SolderWirePad_1x01_Drill1mm, Connector_Wire:SolderWirePad_1x01_Drill1mm, F.Cu at (76.7, 109.7)
- added REF**: SolderWirePad_1x01_Drill1mm, Connector_Wire:SolderWirePad_1x01_Drill1mm, F.Cu at (56.3, 117.3)
- added REF**: SolderWirePad_1x01_Drill1mm, Connector_Wire:SolderWirePad_1x01_Drill1mm, F.Cu at (74.1, 109.7)
- added REF**: SolderWirePad_1x01_Drill1mm, Connector_Wire:SolderWirePad_1x01_Drill1mm, F.Cu at (66.5, 109.7)
- added REF**: SolderWirePad_1x01_Drill1mm, Connector_Wire:SolderWirePad_1x01_Drill1mm, F.Cu at (69.0, 112.2)
- added REF**: SolderWirePad_1x01_Drill1mm, Connector_Wire:SolderWirePad_1x01_Drill1mm, F.Cu at (71.6, 109.7)
- added REF**: SolderWirePad_1x01_Drill1mm, Connector_Wire:SolderWirePad_1x01_Drill1mm, F.Cu at (71.6, 112.2)
- added REF**: SolderWirePad_1x01_Drill1mm, Connector_Wire:SolderWirePad_1x01_Drill1mm, F.Cu at (53.8, 112.2)
- added REF**: SolderWirePad_1x01_Drill1mm, Connector_Wire:SolderWirePad_1x01_Drill1mm, F.Cu at (76.7, 122.4)
- added REF**: SolderWirePad_1x01_Drill1mm, Connector_Wire:SolderWirePad_1x01_Drill1mm, F.Cu at (64.0, 112.2)
- added REF**: SolderWirePad_1x01_Drill1mm, Connector_Wire:SolderWirePad_1x01_Drill1mm, F.Cu at (130.0, 142.7)
- added REF**: SolderWirePad_1x01_Drill1mm, Connector_Wire:SolderWirePad_1x01_Drill1mm, F.Cu at (66.5, 112.2)
- added REF**: SolderWirePad_1x01_Drill1mm, Connector_Wire:SolderWirePad_1x01_Drill1mm, F.Cu at (64.0, 104.6)
- added REF**: SolderWirePad_1x01_Drill1mm, Connector_Wire:SolderWirePad_1x01_Drill1mm, F.Cu at (74.1, 104.6)
- added REF**: SolderWirePad_1x01_Drill1mm, Connector_Wire:SolderWirePad_1x01_Drill1mm, F.Cu at (61.4, 112.2)
- added REF**: SolderWirePad_1x01_Drill1mm, Connector_Wire:SolderWirePad_1x01_Drill1mm, F.Cu at (58.9, 112.2)
- added REF**: SolderWirePad_1x01_Drill1mm, Connector_Wire:SolderWirePad_1x01_Drill1mm, F.Cu at (69.0, 104.6)
- added REF**: SolderWirePad_1x01_Drill1mm, Connector_Wire:SolderWirePad_1x01_Drill1mm, F.Cu at (79.2, 114.8)
- added REF**: SolderWirePad_1x01_Drill1mm, Connector_Wire:SolderWirePad_1x01_Drill1mm, F.Cu at (76.7, 117.3)
- added REF**: SolderWirePad_1x01_Drill1mm, Connector_Wire:SolderWirePad_1x01_Drill1mm, F.Cu at (81.7, 117.3)
- added REF**: SolderWirePad_1x01_Drill1mm, Connector_Wire:SolderWirePad_1x01_Drill1mm, F.Cu at (58.9, 114.8)
- added REF**: SolderWirePad_1x01_Drill1mm, Connector_Wire:SolderWirePad_1x01_Drill1mm, F.Cu at (124.9, 142.7)
- added REF**: SolderWirePad_1x01_Drill1mm, Connector_Wire:SolderWirePad_1x01_Drill1mm, F.Cu at (81.7, 114.8)
- added REF**: SolderWirePad_1x01_Drill1mm, Connector_Wire:SolderWirePad_1x01_Drill1mm, F.Cu at (81.7, 122.4)
- added REF**: SolderWirePad_1x01_Drill1mm, Connector_Wire:SolderWirePad_1x01_Drill1mm, F.Cu at (79.2, 122.4)
- added REF**: SolderWirePad_1x01_Drill1mm, Connector_Wire:SolderWirePad_1x01_Drill1mm, F.Cu at (71.6, 107.2)
- added REF**: SolderWirePad_1x01_Drill1mm, Connector_Wire:SolderWirePad_1x01_Drill1mm, F.Cu at (53.8, 107.2)
- added REF**: SolderWirePad_1x01_Drill1mm, Connector_Wire:SolderWirePad_1x01_Drill1mm, F.Cu at (79.2, 107.2)
- added REF**: SolderWirePad_1x01_Drill1mm, Connector_Wire:SolderWirePad_1x01_Drill1mm, F.Cu at (58.9, 107.2)
- added REF**: SolderWirePad_1x01_Drill1mm, Connector_Wire:SolderWirePad_1x01_Drill1mm, F.Cu at (76.7, 104.6)
- added REF**: SolderWirePad_1x01_Drill1mm, Connector_Wire:SolderWirePad_1x01_Drill1mm, F.Cu at (56.3, 107.2)
- added REF**: SolderWirePad_1x01_Drill1mm, Connector_Wire:SolderWirePad_1x01_Drill1mm, F.Cu at (76.7, 112.2)
- added REF**: SolderWirePad_1x01_Drill1mm, Connector_Wire:SolderWirePad_1x01_Drill1mm, F.Cu at (127.5, 142.7)
- added REF**: SolderWirePad_1x01_Drill1mm, Connector_Wire:SolderWirePad_1x01_Drill1mm, F.Cu at (79.2, 104.6)
- added REF**: SolderWirePad_1x01_Drill1mm, Connector_Wire:SolderWirePad_1x01_Drill1mm, F.Cu at (76.7, 107.2)
- added REF**: SolderWirePad_1x01_Drill1mm, Connector_Wire:SolderWirePad_1x01_Drill1mm, F.Cu at (79.2, 109.7)
- added REF**: SolderWirePad_1x01_Drill1mm, Connector_Wire:SolderWirePad_1x01_Drill1mm, F.Cu at (58.9, 109.7)
- added REF**: SolderWirePad_1x01_Drill1mm, Connector_Wire:SolderWirePad_1x01_Drill1mm, F.Cu at (81.7, 109.7)
- added REF**: SolderWirePad_1x01_Drill1mm, Connector_Wire:SolderWirePad_1x01_Drill1mm, F.Cu at (69.0, 130.0)
- added REF**: SolderWirePad_1x01_Drill1mm, Connector_Wire:SolderWirePad_1x01_Drill1mm, F.Cu at (61.4, 130.0)
- added REF**: SolderWirePad_1x01_Drill1mm, Connector_Wire:SolderWirePad_1x01_Drill1mm, F.Cu at (56.3, 130.0)
- added REF**: SolderWirePad_1x01_Drill1mm, Connector_Wire:SolderWirePad_1x01_Drill1mm, F.Cu at (64.0, 132.6)
- added REF**: SolderWirePad_1x01_Drill1mm, Connector_Wire:SolderWirePad_1x01_Drill1mm, F.Cu at (66.5, 132.6)
- added REF**: SolderWirePad_1x01_Drill1mm, Connector_Wire:SolderWirePad_1x01_Drill1mm, F.Cu at (122.4, 140.2)
- added REF**: SolderWirePad_1x01_Drill1mm, Connector_Wire:SolderWirePad_1x01_Drill1mm, F.Cu at (117.3, 142.7)
- added REF**: SolderWirePad_1x01_Drill1mm, Connector_Wire:SolderWirePad_1x01_Drill1mm, F.Cu at (64.0, 124.9)
- added REF**: SolderWirePad_1x01_Drill1mm, Connector_Wire:SolderWirePad_1x01_Drill1mm, F.Cu at (74.1, 124.9)
- added REF**: SolderWirePad_1x01_Drill1mm, Connector_Wire:SolderWirePad_1x01_Drill1mm, F.Cu at (61.4, 132.6)
- added REF**: SolderWirePad_1x01_Drill1mm, Connector_Wire:SolderWirePad_1x01_Drill1mm, F.Cu at (58.9, 132.6)
- added REF**: SolderWirePad_1x01_Drill1mm, Connector_Wire:SolderWirePad_1x01_Drill1mm, F.Cu at (69.0, 124.9)
- added REF**: SolderWirePad_1x01_Drill1mm, Connector_Wire:SolderWirePad_1x01_Drill1mm, F.Cu at (53.8, 130.0)
- added REF**: SolderWirePad_1x01_Drill1mm, Connector_Wire:SolderWirePad_1x01_Drill1mm, F.Cu at (76.7, 130.0)
- added REF**: SolderWirePad_1x01_Drill1mm, Connector_Wire:SolderWirePad_1x01_Drill1mm, F.Cu at (56.3, 132.6)
- added REF**: SolderWirePad_1x01_Drill1mm, Connector_Wire:SolderWirePad_1x01_Drill1mm, F.Cu at (64.0, 130.0)
- added REF**: SolderWirePad_1x01_Drill1mm, Connector_Wire:SolderWirePad_1x01_Drill1mm, F.Cu at (74.1, 130.0)
- added REF**: SolderWirePad_1x01_Drill1mm, Connector_Wire:SolderWirePad_1x01_Drill1mm, F.Cu at (142.7, 142.7)
- added REF**: SolderWirePad_1x01_Drill1mm, Connector_Wire:SolderWirePad_1x01_Drill1mm, F.Cu at (66.5, 130.0)
- added REF**: SolderWirePad_1x01_Drill1mm, Connector_Wire:SolderWirePad_1x01_Drill1mm, F.Cu at (69.0, 132.6)
- added REF**: SolderWirePad_1x01_Drill1mm, Connector_Wire:SolderWirePad_1x01_Drill1mm, F.Cu at (71.6, 130.0)
- added REF**: SolderWirePad_1x01_Drill1mm, Connector_Wire:SolderWirePad_1x01_Drill1mm, F.Cu at (71.6, 132.6)
- added REF**: SolderWirePad_1x01_Drill1mm, Connector_Wire:SolderWirePad_1x01_Drill1mm, F.Cu at (53.8, 132.6)
- added REF**: SolderWirePad_1x01_Drill1mm, Connector_Wire:SolderWirePad_1x01_Drill1mm, F.Cu at (79.2, 130.0)
- added REF**: SolderWirePad_1x01_Drill1mm, Connector_Wire:SolderWirePad_1x01_Drill1mm, F.Cu at (58.9, 130.0)
- added REF**: SolderWirePad_1x01_Drill1mm, Connector_Wire:SolderWirePad_1x01_Drill1mm, F.Cu at (81.7, 130.0)
- added REF**: SolderWirePad_1x01_Drill1mm, Connector_Wire:SolderWirePad_1x01_Drill1mm, F.Cu at (74.1, 127.5)
- added REF**: SolderWirePad_1x01_Drill1mm, Connector_Wire:SolderWirePad_1x01_Drill1mm, F.Cu at (74.1, 132.6)
- added REF**: SolderWirePad_1x01_Drill1mm, Connector_Wire:SolderWirePad_1x01_Drill1mm, F.Cu at (122.4, 142.7)
- added REF**: SolderWirePad_1x01_Drill1mm, Connector_Wire:SolderWirePad_1x01_Drill1mm, F.Cu at (56.3, 124.9)
- added REF**: SolderWirePad_1x01_Drill1mm, Connector_Wire:SolderWirePad_1x01_Drill1mm, F.Cu at (64.0, 127.5)
- added REF**: SolderWirePad_1x01_Drill1mm, Connector_Wire:SolderWirePad_1x01_Drill1mm, F.Cu at (66.5, 127.5)
- added REF**: SolderWirePad_1x01_Drill1mm, Connector_Wire:SolderWirePad_1x01_Drill1mm, F.Cu at (61.4, 127.5)
- added REF**: SolderWirePad_1x01_Drill1mm, Connector_Wire:SolderWirePad_1x01_Drill1mm, F.Cu at (61.4, 124.9)
- added REF**: SolderWirePad_1x01_Drill1mm, Connector_Wire:SolderWirePad_1x01_Drill1mm, F.Cu at (66.5, 124.9)
- added REF**: SolderWirePad_1x01_Drill1mm, Connector_Wire:SolderWirePad_1x01_Drill1mm, F.Cu at (69.0, 127.5)
- added REF**: SolderWirePad_1x01_Drill1mm, Connector_Wire:SolderWirePad_1x01_Drill1mm, F.Cu at (71.6, 124.9)
- added REF**: SolderWirePad_1x01_Drill1mm, Connector_Wire:SolderWirePad_1x01_Drill1mm, F.Cu at (71.6, 127.5)
- added REF**: SolderWirePad_1x01_Drill1mm, Connector_Wire:SolderWirePad_1x01_Drill1mm, F.Cu at (53.8, 127.5)
- added REF**: SolderWirePad_1x01_Drill1mm, Connector_Wire:SolderWirePad_1x01_Drill1mm, F.Cu at (119.9, 142.7)
- added REF**: SolderWirePad_1x01_Drill1mm, Connector_Wire:SolderWirePad_1x01_Drill1mm, F.Cu at (79.2, 127.5)
- added REF**: SolderWirePad_1x01_Drill1mm, Connector_Wire:SolderWirePad_1x01_Drill1mm, F.Cu at (58.9, 127.5)
- added REF**: SolderWirePad_1x01_Drill1mm, Connector_Wire:SolderWirePad_1x01_Drill1mm, F.Cu at (53.8, 124.9)
- added REF**: SolderWirePad_1x01_Drill1mm, Connector_Wire:SolderWirePad_1x01_Drill1mm, F.Cu at (76.7, 124.9)
- added REF**: SolderWirePad_1x01_Drill1mm, Connector_Wire:SolderWirePad_1x01_Drill1mm, F.Cu at (56.3, 127.5)
- added REF**: SolderWirePad_1x01_Drill1mm, Connector_Wire:SolderWirePad_1x01_Drill1mm, F.Cu at (76.7, 132.6)
- added REF**: SolderWirePad_1x01_Drill1mm, Connector_Wire:SolderWirePad_1x01_Drill1mm, F.Cu at (79.2, 124.9)
- added REF**: SolderWirePad_1x01_Drill1mm, Connector_Wire:SolderWirePad_1x01_Drill1mm, F.Cu at (76.7, 127.5)
- added REF**: SolderWirePad_1x01_Drill1mm, Connector_Wire:SolderWirePad_1x01_Drill1mm, F.Cu at (81.7, 127.5)
- added REF**: SolderWirePad_1x01_Drill1mm, Connector_Wire:SolderWirePad_1x01_Drill1mm, F.Cu at (58.9, 124.9)
- added REF**: SolderWirePad_1x01_Drill1mm, Connector_Wire:SolderWirePad_1x01_Drill1mm, F.Cu at (114.8, 145.3)
- added REF**: SolderWirePad_1x01_Drill1mm, Connector_Wire:SolderWirePad_1x01_Drill1mm, F.Cu at (81.7, 124.9)
- added REF**: SolderWirePad_1x01_Drill1mm, Connector_Wire:SolderWirePad_1x01_Drill1mm, F.Cu at (81.7, 132.6)
- added REF**: SolderWirePad_1x01_Drill1mm, Connector_Wire:SolderWirePad_1x01_Drill1mm, F.Cu at (79.2, 132.6)
- added REF**: SolderWirePad_1x01_Drill1mm, Connector_Wire:SolderWirePad_1x01_Drill1mm, F.Cu at (69.0, 135.1)
- added REF**: SolderWirePad_1x01_Drill1mm, Connector_Wire:SolderWirePad_1x01_Drill1mm, F.Cu at (61.4, 135.1)
- added REF**: SolderWirePad_1x01_Drill1mm, Connector_Wire:SolderWirePad_1x01_Drill1mm, F.Cu at (56.3, 135.1)
- added REF**: SolderWirePad_1x01_Drill1mm, Connector_Wire:SolderWirePad_1x01_Drill1mm, F.Cu at (64.0, 137.6)
- added REF**: SolderWirePad_1x01_Drill1mm, Connector_Wire:SolderWirePad_1x01_Drill1mm, F.Cu at (66.5, 137.6)
- added REF**: SolderWirePad_1x01_Drill1mm, Connector_Wire:SolderWirePad_1x01_Drill1mm, F.Cu at (61.4, 137.6)
- added REF**: SolderWirePad_1x01_Drill1mm, Connector_Wire:SolderWirePad_1x01_Drill1mm, F.Cu at (58.9, 137.6)
- added REF**: SolderWirePad_1x01_Drill1mm, Connector_Wire:SolderWirePad_1x01_Drill1mm, F.Cu at (117.3, 145.3)
- added REF**: SolderWirePad_1x01_Drill1mm, Connector_Wire:SolderWirePad_1x01_Drill1mm, F.Cu at (53.8, 135.1)
- added REF**: SolderWirePad_1x01_Drill1mm, Connector_Wire:SolderWirePad_1x01_Drill1mm, F.Cu at (76.7, 135.1)
- added REF**: SolderWirePad_1x01_Drill1mm, Connector_Wire:SolderWirePad_1x01_Drill1mm, F.Cu at (56.3, 137.6)
- added REF**: SolderWirePad_1x01_Drill1mm, Connector_Wire:SolderWirePad_1x01_Drill1mm, F.Cu at (64.0, 135.1)
- added REF**: SolderWirePad_1x01_Drill1mm, Connector_Wire:SolderWirePad_1x01_Drill1mm, F.Cu at (74.1, 135.1)
- added REF**: SolderWirePad_1x01_Drill1mm, Connector_Wire:SolderWirePad_1x01_Drill1mm, F.Cu at (66.5, 135.1)
- added REF**: SolderWirePad_1x01_Drill1mm, Connector_Wire:SolderWirePad_1x01_Drill1mm, F.Cu at (69.0, 137.6)
- added REF**: SolderWirePad_1x01_Drill1mm, Connector_Wire:SolderWirePad_1x01_Drill1mm, F.Cu at (71.6, 135.1)
- added REF**: SolderWirePad_1x01_Drill1mm, Connector_Wire:SolderWirePad_1x01_Drill1mm, F.Cu at (71.6, 137.6)
- added REF**: SolderWirePad_1x01_Drill1mm, Connector_Wire:SolderWirePad_1x01_Drill1mm, F.Cu at (53.8, 137.6)
- added REF**: SolderWirePad_1x01_Drill1mm, Connector_Wire:SolderWirePad_1x01_Drill1mm, F.Cu at (130.0, 145.3)
- added REF**: SolderWirePad_1x01_Drill1mm, Connector_Wire:SolderWirePad_1x01_Drill1mm, F.Cu at (79.2, 135.1)
- added REF**: SolderWirePad_1x01_Drill1mm, Connector_Wire:SolderWirePad_1x01_Drill1mm, F.Cu at (58.9, 135.1)
- added REF**: SolderWirePad_1x01_Drill1mm, Connector_Wire:SolderWirePad_1x01_Drill1mm, F.Cu at (81.7, 135.1)
- added REF**: SolderWirePad_1x01_Drill1mm, Connector_Wire:SolderWirePad_1x01_Drill1mm, F.Cu at (74.1, 137.6)
- added REF**: SolderWirePad_1x01_Drill1mm, Connector_Wire:SolderWirePad_1x01_Drill1mm, F.Cu at (76.7, 137.6)
- added REF**: SolderWirePad_1x01_Drill1mm, Connector_Wire:SolderWirePad_1x01_Drill1mm, F.Cu at (81.7, 137.6)
- added REF**: SolderWirePad_1x01_Drill1mm, Connector_Wire:SolderWirePad_1x01_Drill1mm, F.Cu at (79.2, 137.6)
- added REF**: SolderWirePad_1x01_Drill1mm, Connector_Wire:SolderWirePad_1x01_Drill1mm, F.Cu at (64.0, 140.2)
- added REF**: SolderWirePad_1x01_Drill1mm, Connector_Wire:SolderWirePad_1x01_Drill1mm, F.Cu at (66.5, 140.2)
- added REF**: SolderWirePad_1x01_Drill1mm, Connector_Wire:SolderWirePad_1x01_Drill1mm, F.Cu at (61.4, 140.2)
- added REF**: SolderWirePad_1x01_Drill1mm, Connector_Wire:SolderWirePad_1x01_Drill1mm, F.Cu at (124.9, 145.3)
- added REF**: SolderWirePad_1x01_Drill1mm, Connector_Wire:SolderWirePad_1x01_Drill1mm, F.Cu at (58.9, 140.2)
- added REF**: SolderWirePad_1x01_Drill1mm, Connector_Wire:SolderWirePad_1x01_Drill1mm, F.Cu at (56.3, 140.2)
- added REF**: SolderWirePad_1x01_Drill1mm, Connector_Wire:SolderWirePad_1x01_Drill1mm, F.Cu at (69.0, 140.2)
- added REF**: SolderWirePad_1x01_Drill1mm, Connector_Wire:SolderWirePad_1x01_Drill1mm, F.Cu at (71.6, 140.2)
- added REF**: SolderWirePad_1x01_Drill1mm, Connector_Wire:SolderWirePad_1x01_Drill1mm, F.Cu at (53.8, 140.2)
- added REF**: SolderWirePad_1x01_Drill1mm, Connector_Wire:SolderWirePad_1x01_Drill1mm, F.Cu at (74.1, 140.2)
- added REF**: SolderWirePad_1x01_Drill1mm, Connector_Wire:SolderWirePad_1x01_Drill1mm, F.Cu at (76.7, 140.2)
- added REF**: SolderWirePad_1x01_Drill1mm, Connector_Wire:SolderWirePad_1x01_Drill1mm, F.Cu at (81.7, 140.2)
- added REF**: SolderWirePad_1x01_Drill1mm, Connector_Wire:SolderWirePad_1x01_Drill1mm, F.Cu at (79.2, 140.2)
- added REF**: SolderWirePad_1x01_Drill1mm, Connector_Wire:SolderWirePad_1x01_Drill1mm, F.Cu at (81.7, 142.7)
- added REF**: SolderWirePad_1x01_Drill1mm, Connector_Wire:SolderWirePad_1x01_Drill1mm, F.Cu at (127.5, 145.3)
- added REF**: SolderWirePad_1x01_Drill1mm, Connector_Wire:SolderWirePad_1x01_Drill1mm, F.Cu at (79.2, 142.7)
- added REF**: SolderWirePad_1x01_Drill1mm, Connector_Wire:SolderWirePad_1x01_Drill1mm, F.Cu at (76.7, 142.7)
- added REF**: SolderWirePad_1x01_Drill1mm, Connector_Wire:SolderWirePad_1x01_Drill1mm, F.Cu at (74.1, 142.7)
- added REF**: SolderWirePad_1x01_Drill1mm, Connector_Wire:SolderWirePad_1x01_Drill1mm, F.Cu at (71.6, 142.7)
- added REF**: SolderWirePad_1x01_Drill1mm, Connector_Wire:SolderWirePad_1x01_Drill1mm, F.Cu at (69.0, 142.7)
- added REF**: SolderWirePad_1x01_Drill1mm, Connector_Wire:SolderWirePad_1x01_Drill1mm, F.Cu at (66.5, 142.7)
- added REF**: SolderWirePad_1x01_Drill1mm, Connector_Wire:SolderWirePad_1x01_Drill1mm, F.Cu at (64.0, 142.7)
- added REF**: SolderWirePad_1x01_Drill1mm, Connector_Wire:SolderWirePad_1x01_Drill1mm, F.Cu at (61.4, 142.7)
- added REF**: SolderWirePad_1x01_Drill1mm, Connector_Wire:SolderWirePad_1x01_Drill1mm, F.Cu at (58.9, 142.7)
- added REF**: SolderWirePad_1x01_Drill1mm, Connector_Wire:SolderWirePad_1x01_Drill1mm, F.Cu at (56.3, 142.7)
- added REF**: SolderWirePad_1x01_Drill1mm, Connector_Wire:SolderWirePad_1x01_Drill1mm, F.Cu at (142.7, 145.3)
- added REF**: SolderWirePad_1x01_Drill1mm, Connector_Wire:SolderWirePad_1x01_Drill1mm, F.Cu at (127.5, 140.2)
- added REF**: SolderWirePad_1x01_Drill1mm, Connector_Wire:SolderWirePad_1x01_Drill1mm, F.Cu at (122.4, 145.3)
- added REF**: SolderWirePad_1x01_Drill1mm, Connector_Wire:SolderWirePad_1x01_Drill1mm, F.Cu at (53.8, 142.7)
- added REF**: SolderWirePad_1x01_Drill1mm, Connector_Wire:SolderWirePad_1x01_Drill1mm, F.Cu at (112.2, 145.3)
- added REF**: SolderWirePad_1x01_Drill1mm, Connector_Wire:SolderWirePad_1x01_Drill1mm, F.Cu at (119.9, 145.3)
- added REF**: SolderWirePad_1x01_Drill1mm, Connector_Wire:SolderWirePad_1x01_Drill1mm, F.Cu at (132.6, 145.3)
- added REF**: SolderWirePad_1x01_Drill1mm, Connector_Wire:SolderWirePad_1x01_Drill1mm, F.Cu at (140.2, 145.3)
- added REF**: SolderWirePad_1x01_Drill1mm, Connector_Wire:SolderWirePad_1x01_Drill1mm, F.Cu at (135.1, 145.3)
- added REF**: SolderWirePad_1x01_Drill1mm, Connector_Wire:SolderWirePad_1x01_Drill1mm, F.Cu at (137.6, 145.3)
- added REF**: SolderWirePad_1x01_Drill1mm, Connector_Wire:SolderWirePad_1x01_Drill1mm, F.Cu at (109.7, 147.8)
- added REF**: SolderWirePad_1x01_Drill1mm, Connector_Wire:SolderWirePad_1x01_Drill1mm, F.Cu at (122.4, 147.8)
- added REF**: SolderWirePad_1x01_Drill1mm, Connector_Wire:SolderWirePad_1x01_Drill1mm, F.Cu at (112.2, 147.8)
- added REF**: SolderWirePad_1x01_Drill1mm, Connector_Wire:SolderWirePad_1x01_Drill1mm, F.Cu at (119.9, 140.2)
- added REF**: SolderWirePad_1x01_Drill1mm, Connector_Wire:SolderWirePad_1x01_Drill1mm, F.Cu at (119.9, 147.8)
- added REF**: SolderWirePad_1x01_Drill1mm, Connector_Wire:SolderWirePad_1x01_Drill1mm, F.Cu at (114.8, 147.8)
- added REF**: SolderWirePad_1x01_Drill1mm, Connector_Wire:SolderWirePad_1x01_Drill1mm, F.Cu at (117.3, 147.8)
- added REF**: SolderWirePad_1x01_Drill1mm, Connector_Wire:SolderWirePad_1x01_Drill1mm, F.Cu at (132.6, 147.8)
- added REF**: SolderWirePad_1x01_Drill1mm, Connector_Wire:SolderWirePad_1x01_Drill1mm, F.Cu at (130.0, 147.8)
- added REF**: SolderWirePad_1x01_Drill1mm, Connector_Wire:SolderWirePad_1x01_Drill1mm, F.Cu at (124.9, 147.8)
- added REF**: SolderWirePad_1x01_Drill1mm, Connector_Wire:SolderWirePad_1x01_Drill1mm, F.Cu at (127.5, 147.8)
- added REF**: SolderWirePad_1x01_Drill1mm, Connector_Wire:SolderWirePad_1x01_Drill1mm, F.Cu at (135.1, 147.8)
- added REF**: SolderWirePad_1x01_Drill1mm, Connector_Wire:SolderWirePad_1x01_Drill1mm, F.Cu at (137.6, 147.8)
- added REF**: SolderWirePad_1x01_Drill1mm, Connector_Wire:SolderWirePad_1x01_Drill1mm, F.Cu at (140.2, 147.8)
- added REF**: SolderWirePad_1x01_Drill1mm, Connector_Wire:SolderWirePad_1x01_Drill1mm, F.Cu at (142.7, 140.2)
- added REF**: SolderWirePad_1x01_Drill1mm, Connector_Wire:SolderWirePad_1x01_Drill1mm, F.Cu at (142.7, 147.8)
- added REF**: SolderWirePad_1x01_Drill1mm, Connector_Wire:SolderWirePad_1x01_Drill1mm, F.Cu at (53.8, 104.6)
- added REF**: SolderWirePad_1x01_Drill1mm, Connector_Wire:SolderWirePad_1x01_Drill1mm, F.Cu at (74.1, 99.5)
- added REF**: SolderWirePad_1x01_Drill1mm, Connector_Wire:SolderWirePad_1x01_Drill1mm, F.Cu at (79.2, 99.5)
- added REF**: SolderWirePad_1x01_Drill1mm, Connector_Wire:SolderWirePad_1x01_Drill1mm, F.Cu at (53.8, 99.5)
- added REF**: SolderWirePad_1x01_Drill1mm, Connector_Wire:SolderWirePad_1x01_Drill1mm, F.Cu at (76.7, 99.5)
- added REF**: SolderWirePad_1x01_Drill1mm, Connector_Wire:SolderWirePad_1x01_Drill1mm, F.Cu at (58.9, 99.5)
- added REF**: SolderWirePad_1x01_Drill1mm, Connector_Wire:SolderWirePad_1x01_Drill1mm, F.Cu at (81.7, 99.5)
- added REF**: SolderWirePad_1x01_Drill1mm, Connector_Wire:SolderWirePad_1x01_Drill1mm, F.Cu at (56.3, 99.5)
- added REF**: SolderWirePad_1x01_Drill1mm, Connector_Wire:SolderWirePad_1x01_Drill1mm, F.Cu at (66.5, 99.5)
- added REF**: SolderWirePad_1x01_Drill1mm, Connector_Wire:SolderWirePad_1x01_Drill1mm, F.Cu at (140.2, 140.2)
- added REF**: SolderWirePad_1x01_Drill1mm, Connector_Wire:SolderWirePad_1x01_Drill1mm, F.Cu at (61.4, 99.5)
- added REF**: SolderWirePad_1x01_Drill1mm, Connector_Wire:SolderWirePad_1x01_Drill1mm, F.Cu at (71.6, 99.5)
- added REF**: SolderWirePad_1x01_Drill1mm, Connector_Wire:SolderWirePad_1x01_Drill1mm, F.Cu at (69.0, 99.5)
- added REF**: SolderWirePad_1x01_Drill1mm, Connector_Wire:SolderWirePad_1x01_Drill1mm, F.Cu at (64.0, 99.5)
- added REF**: SolderWirePad_1x01_Drill1mm, Connector_Wire:SolderWirePad_1x01_Drill1mm, F.Cu at (91.9, 142.7)
- added REF**: SolderWirePad_1x01_Drill1mm, Connector_Wire:SolderWirePad_1x01_Drill1mm, F.Cu at (89.4, 140.2)
- added REF**: SolderWirePad_1x01_Drill1mm, Connector_Wire:SolderWirePad_1x01_Drill1mm, F.Cu at (89.4, 142.7)
- added REF**: SolderWirePad_1x01_Drill1mm, Connector_Wire:SolderWirePad_1x01_Drill1mm, F.Cu at (89.4, 145.3)
- added REF**: SolderWirePad_1x01_Drill1mm, Connector_Wire:SolderWirePad_1x01_Drill1mm, F.Cu at (89.4, 147.8)
- added REF**: SolderWirePad_1x01_Drill1mm, Connector_Wire:SolderWirePad_1x01_Drill1mm, F.Cu at (86.8, 147.8)
- added REF**: SolderWirePad_1x01_Drill1mm, Connector_Wire:SolderWirePad_1x01_Drill1mm, F.Cu at (135.1, 140.2)
- added REF**: SolderWirePad_1x01_Drill1mm, Connector_Wire:SolderWirePad_1x01_Drill1mm, F.Cu at (86.8, 145.3)
- added REF**: SolderWirePad_1x01_Drill1mm, Connector_Wire:SolderWirePad_1x01_Drill1mm, F.Cu at (86.8, 140.2)
- added REF**: SolderWirePad_1x01_Drill1mm, Connector_Wire:SolderWirePad_1x01_Drill1mm, F.Cu at (86.8, 137.6)
- added REF**: SolderWirePad_1x01_Drill1mm, Connector_Wire:SolderWirePad_1x01_Drill1mm, F.Cu at (86.8, 142.7)
- added REF**: SolderWirePad_1x01_Drill1mm, Connector_Wire:SolderWirePad_1x01_Drill1mm, F.Cu at (84.3, 135.1)
- added REF**: SolderWirePad_1x01_Drill1mm, Connector_Wire:SolderWirePad_1x01_Drill1mm, F.Cu at (84.3, 145.3)
- added REF**: SolderWirePad_1x01_Drill1mm, Connector_Wire:SolderWirePad_1x01_Drill1mm, F.Cu at (84.3, 140.2)
- added REF**: SolderWirePad_1x01_Drill1mm, Connector_Wire:SolderWirePad_1x01_Drill1mm, F.Cu at (84.3, 147.8)
- added REF**: SolderWirePad_1x01_Drill1mm, Connector_Wire:SolderWirePad_1x01_Drill1mm, F.Cu at (84.3, 137.6)
- added REF**: SolderWirePad_1x01_Drill1mm, Connector_Wire:SolderWirePad_1x01_Drill1mm, F.Cu at (84.3, 142.7)
- added REF**: SolderWirePad_1x01_Drill1mm, Connector_Wire:SolderWirePad_1x01_Drill1mm, F.Cu at (137.6, 140.2)
- added REF**: SolderWirePad_1x01_Drill1mm, Connector_Wire:SolderWirePad_1x01_Drill1mm, F.Cu at (79.2, 147.8)
- added REF**: SolderWirePad_1x01_Drill1mm, Connector_Wire:SolderWirePad_1x01_Drill1mm, F.Cu at (61.4, 147.8)
- added REF**: SolderWirePad_1x01_Drill1mm, Connector_Wire:SolderWirePad_1x01_Drill1mm, F.Cu at (66.5, 147.8)
- added REF**: SolderWirePad_1x01_Drill1mm, Connector_Wire:SolderWirePad_1x01_Drill1mm, F.Cu at (69.0, 147.8)
- added REF**: SolderWirePad_1x01_Drill1mm, Connector_Wire:SolderWirePad_1x01_Drill1mm, F.Cu at (64.0, 147.8)
- added REF**: SolderWirePad_1x01_Drill1mm, Connector_Wire:SolderWirePad_1x01_Drill1mm, F.Cu at (71.6, 147.8)
- added REF**: SolderWirePad_1x01_Drill1mm, Connector_Wire:SolderWirePad_1x01_Drill1mm, F.Cu at (74.1, 147.8)
- added REF**: SolderWirePad_1x01_Drill1mm, Connector_Wire:SolderWirePad_1x01_Drill1mm, F.Cu at (76.7, 147.8)
- added REF**: SolderWirePad_1x01_Drill1mm, Connector_Wire:SolderWirePad_1x01_Drill1mm, F.Cu at (81.7, 147.8)
- added REF**: SolderWirePad_1x01_Drill1mm, Connector_Wire:SolderWirePad_1x01_Drill1mm, F.Cu at (58.9, 147.8)
- added REF**: SolderWirePad_1x01_Drill1mm, Connector_Wire:SolderWirePad_1x01_Drill1mm, F.Cu at (132.6, 140.2)
- added REF**: SolderWirePad_1x01_Drill1mm, Connector_Wire:SolderWirePad_1x01_Drill1mm, F.Cu at (64.0, 145.3)
- added REF**: SolderWirePad_1x01_Drill1mm, Connector_Wire:SolderWirePad_1x01_Drill1mm, F.Cu at (66.5, 145.3)
- added REF**: SolderWirePad_1x01_Drill1mm, Connector_Wire:SolderWirePad_1x01_Drill1mm, F.Cu at (61.4, 145.3)
- added REF**: SolderWirePad_1x01_Drill1mm, Connector_Wire:SolderWirePad_1x01_Drill1mm, F.Cu at (58.9, 145.3)
- added REF**: SolderWirePad_1x01_Drill1mm, Connector_Wire:SolderWirePad_1x01_Drill1mm, F.Cu at (69.0, 145.3)
- added REF**: SolderWirePad_1x01_Drill1mm, Connector_Wire:SolderWirePad_1x01_Drill1mm, F.Cu at (71.6, 145.3)
- added REF**: SolderWirePad_1x01_Drill1mm, Connector_Wire:SolderWirePad_1x01_Drill1mm, F.Cu at (74.1, 145.3)
- added REF**: SolderWirePad_1x01_Drill1mm, Connector_Wire:SolderWirePad_1x01_Drill1mm, F.Cu at (76.7, 145.3)
- added REF**: SolderWirePad_1x01_Drill1mm, Connector_Wire:SolderWirePad_1x01_Drill1mm, F.Cu at (81.7, 145.3)
- added REF**: SolderWirePad_1x01_Drill1mm, Connector_Wire:SolderWirePad_1x01_Drill1mm, F.Cu at (79.2, 145.3)
Routing:
- net -12V: track 7.62 -> 128.2 mm
- net +3V3: track 34.8 -> 144.4 mm, vias 0 -> 1
- net +5VD: track 17.6 -> 100.0 mm, vias 0 -> 3
- net VEE: track 16.9 -> 52.2 mm
- net (no net): track 0.00 -> 15.3 mm
- net +5V: track 100.2 -> 85.7 mm, vias 0 -> 138
- net GND: track 205.7 -> 211.0 mm, vias 0 -> 118
- net /PWR_OK: track 56.9 -> 57.6 mm, vias 0 -> 3
- added copper zone on F.Cu, net (none)
- added copper zone on B.Cu, net +5V
- added copper zone on F.Cu, net +5V
- added copper zone on B.Cu, net GND
Other:
- outline, holes or cut-outs redrawn
- board text added: "3V3"
- board text added: "5V0"
- board text added: "GND"
- board text added: "RPiCluster2/Motherboard © 2018 Sugizaki Yukimasa"
